Commit message: created inertial xacro and made updates in core xacro

File: description/robot_core.xacro (robot description, xacro)
@@ -1,5 +1,5 @@
 <?xml version="1.0"?>
 <robot xmlns:xacro="http://www.ros.org/wiki/xacro">
-  <!-- Define materials -->
+  <xacro:include filename="inertial_macros.xacro" />
   <material name="white">
     <color rgba="1 1 1 1" />
@@ -38,4 +38,7 @@
       </geometry>
     </collision>
+    <xacro:inertial_box mass="0.5" x="0.6" y="0.4" z="0.2">
+      <origin xyz="0.3 0 0.1" rpy="0 0 0" />
+    </xacro:inertial_box>
   </link>
   <!-- Left wheel joint and link -->
@@ -58,4 +61,7 @@
       </geometry>
     </collision>
+    <xacro:inertial_cylinder mass="0.1" length="0.05" radius="0.1">
+      <origin xyz="0 0 0" rpy="0 0 0" />
+    </xacro:inertial_cylinder>
   </link>
   <!-- Right wheel joint and link -->
@@ -78,27 +84,33 @@
       </geometry>
     </collision>
-  </link>
- <!--Caster wheel joints and links-->
+    <xacro:inertial_cylinder mass="0.1" length="0.05" radius="0.1">
+      <origin xyz="0 0 0" rpy="0 0 0" />
+    </xacro:inertial_cylinder>
+  </link>
+  <!-- Caster wheels -->
   <joint name="caster_wheel_1_joint" type="fixed">
-    <parent link="chassis"/>
-    <child link="caster_wheel_1"/>
-    <origin xyz="0.1 0.11 0"/>
+    <parent link="chassis" />
+    <child link="caster_wheel_1" />
+    <origin xyz="0.1 0.11 0" />
   </joint>
   <link name="caster_wheel_1">
     <visual>
       <geometry>
-        <sphere radius="0.09"/>
-      </geometry>
-      <material name="black"/>
-    </visual>
-    <collision>
-      <geometry>
-        <sphere radius="0.09"/>
-      </geometry>
-    </collision>
+        <sphere radius="0.09" />
+      </geometry>
+      <material name="black" />
+    </visual>
+    <collision>
+      <geometry>
+        <sphere radius="0.09" />
+      </geometry>
+    </collision>
+    <xacro:inertial_sphere mass="0.1" radius="0.09">
+      <origin xyz="0 0 0" rpy="0 0 0" />
+    </xacro:inertial_sphere>
   </link>
   <joint name="caster_wheel_2_joint" type="fixed">
-    <parent link="chassis"/>
-    <child link="caster_wheel_2"/>
+    <parent link="chassis" />
+    <child link="caster_wheel_2" />
     <origin xyz="0.1 -0.11 0" />
   </joint>
@@ -106,51 +118,60 @@
     <visual>
       <geometry>
-        <sphere radius="0.09"/>
-      </geometry>
-      <material name="black"/>
-    </visual>
-    <collision>
-      <geometry>
-        <sphere radius="0.09"/>
-      </geometry>
-    </collision>
+        <sphere radius="0.09" />
+      </geometry>
+      <material name="black" />
+    </visual>
+    <collision>
+      <geometry>
+        <sphere radius="0.09" />
+      </geometry>
+    </collision>
+    <xacro:inertial_sphere mass="0.1" radius="0.09">
+      <origin xyz="0 0 0" rpy="0 0 0" />
+    </xacro:inertial_sphere>
   </link>
   <joint name="base_caster_wheel_3_joint" type="fixed">
-    <parent link="base_link"/>
-    <child link="caster_wheel_3"/>
-    <origin xyz="0.4 0.11 0" rpy="0 0 0"/>
+    <parent link="base_link" />
+    <child link="caster_wheel_3" />
+    <origin xyz="0.4 0.11 0" rpy="0 0 0" />
   </joint>
   <link name="caster_wheel_3">
     <visual>
       <geometry>
-        <sphere radius="0.09"/>
-      </geometry>
-      <material name="black"/>
-    </visual>
-    <collision>
-      <geometry>
-        <sphere radius="0.09"/>
-      </geometry>
-    </collision>
+        <sphere radius="0.09" />
+      </geometry>
+      <material name="black" />
+    </visual>
+    <collision>
+      <geometry>
+        <sphere radius="0.09" />
+      </geometry>
+    </collision>
+    <xacro:inertial_sphere mass="0.1" radius="0.09">
+      <origin xyz="0 0 0" rpy="0 0 0" />
+    </xacro:inertial_sphere>
   </link>
   <joint name="base_caster_wheel_4_joint" type="fixed">
-    <parent link="base_link"/>
-    <child link="caster_wheel_4"/>
-    <origin xyz="0.4 -0.11 0" rpy="0 0 0"/>
+    <parent link="base_link" />
+    <child link="caster_wheel_4" />
+    <origin xyz="0.4 -0.11 0" rpy="0 0 0" />
   </joint>
   <link name="caster_wheel_4">
     <visual>
       <geometry>
-        <sphere radius="0.09"/>
-      </geometry>
-      <material name="black"/>
-    </visual>
-    <collision>
-      <geometry>
-        <sphere radius="0.09"/>
-      </geometry>
-    </collision>
-  </link>
- <!--LiDAR Tower joint and  Link-->
+        <sphere radius="0.09" />
+      </geometry>
+      <material name="black" />
+    </visual>
+    <collision>
+      <geometry>
+        <sphere radius="0.09" />
+      </geometry>
+    </collision>
+    <xacro:inertial_sphere mass="0.1" radius="0.09">
+      <origin xyz="0 0 0" rpy="0 0 0" />
+    </xacro:inertial_sphere>
+  </link>
+  <!-- LiDAR Tower -->
   <joint name="base_LiDAR_Tower_joint" type="fixed">
     <parent link="chassis" />
@@ -161,34 +182,40 @@
     <visual>
       <geometry>
-        <box size="0.085 0.085 0.15"/>
-      </geometry>
-      <material name="orange"/>
-    </visual>
-    <collision>
-      <geometry>
-        <box size="0.085 0.085 0.15"/>
-      </geometry>
-    </collision>
-  </link>
-<!-- LiDAR joint and Link-->
+        <box size="0.085 0.085 0.15" />
+      </geometry>
+      <material name="orange" />
+    </visual>
+    <collision>
+      <geometry>
+        <box size="0.085 0.085 0.15" />
+      </geometry>
+    </collision>
+    <xacro:inertial_box mass="0.1" x="0.085" y="0.085" z="0.15">
+      <origin xyz="0 0 0" rpy="0 0 0" />
+    </xacro:inertial_box>
+  </link>
+  <!-- LiDAR Sensor -->
   <joint name="LiDAR_Tower_to_LiDAR_joint" type="fixed">
-    <parent link="LiDAR_Tower"/>
-    <child link="LiDAR"/>
-    <origin xyz="0 0 0" rpy="0 0 0"/>
+    <parent link="LiDAR_Tower" />
+    <child link="LiDAR" />
+    <origin xyz="0 0 0" rpy="0 0 0" />
   </joint>
   <link name="LiDAR">
     <visual>
       <geometry>
-        <cylinder radius="0.05" length="0.02"/>
-      </geometry>
-      <origin xyz="0 0 0.085" rpy="0 0 0"/>
-      <material name="black"/>
-    </visual>
-    <collision>
-      <geometry>
-        <cylinder radius="0.05" length="0.02"/>
-      </geometry>
-      <origin xyz="0 0 0.085" rpy="0 0 0"/>
-    </collision>
+        <cylinder radius="0.05" length="0.02" />
+      </geometry>
+      <origin xyz="0 0 0.085" rpy="0 0 0" />
+      <material name="black" />
+    </visual>
+    <collision>
+      <geometry>
+        <cylinder radius="0.05" length="0.02" />
+      </geometry>
+      <origin xyz="0 0 0.085" rpy="0 0 0" />
+    </collision>
+    <xacro:inertial_cylinder mass="0.1" length="0.02" radius="0.05">
+      <origin xyz="0 0 0" rpy="0 0 0" />
+    </xacro:inertial_cylinder>
   </link>
 </robot>
