Commit message: small changes

File: description/robot.urdf.xacro (robot description, xacro)
@@ -2,3 +2,4 @@
 <robot xmlns:xacro="http://www.ros.org/wiki/xacro" name="robot" >
     <xacro:include filename="robot_core.xacro" />
+    <xacro:include filename="gazebo_control.xacro" />
 </robot>

File: description/robot_core.xacro (robot description, xacro)
@@ -26,25 +26,28 @@
   <link name="chassis">
     <visual>
-      <origin xyz="0.3 0 0.1" />
+      <origin xyz="0.15 0 0.075" />
       <geometry>
-        <box size="0.6 0.4 0.2" />
+        <box size="0.3 0.3 0.15" />
       </geometry>
       <material name="white" />
     </visual>
     <collision>
-      <origin xyz="0.3 0 0.1" />
+      <origin xyz="0.15 0 0.075" />
       <geometry>
-        <box size="0.6 0.4 0.2" />
+        <box size="0.3 0.3 0.15" />
       </geometry>
     </collision>
-    <xacro:inertial_box mass="0.5" x="0.6" y="0.4" z="0.2">
-      <origin xyz="0.3 0 0.1" rpy="0 0 0" />
+    <xacro:inertial_box mass="0.5" x="0.3" y="0.3" z="0.15">
+      <origin xyz="0.15 0 0.075" rpy="0 0 0" />
     </xacro:inertial_box>
   </link>
+  <gazebo reference="chassis">
+    <material>Gazebo/White</material>
+  </gazebo>
   <!-- Left wheel joint and link -->
   <joint name="left_wheel_joint" type="continuous">
     <parent link="base_link" />
     <child link="left_wheel" />
-    <origin xyz="0.20 0.225 0" rpy="-${pi/2} 0 0" />
+    <origin xyz="0.0 0.175 0" rpy="-${pi/2} 0 0" />
     <axis xyz="0 0 1" />
   </joint>
@@ -52,5 +55,5 @@
     <visual>
       <geometry>
-        <cylinder radius="0.1" length="0.05" />
+        <cylinder radius="0.05" length="0.04" />
       </geometry>
       <material name="blue" />
@@ -58,22 +61,25 @@
     <collision>
       <geometry>
-        <cylinder radius="0.1" length="0.05" />
+        <cylinder radius="0.05" length="0.04" />
       </geometry>
     </collision>
-    <xacro:inertial_cylinder mass="0.1" length="0.05" radius="0.1">
+    <xacro:inertial_cylinder mass="0.1" length="0.04" radius="0.05">
       <origin xyz="0 0 0" rpy="0 0 0" />
     </xacro:inertial_cylinder>
   </link>
+  <gazebo reference="left_wheel">
+    <material>Gazebo/Blue</material>
+  </gazebo>
   <!-- Right wheel joint and link -->
   <joint name="right_wheel_joint" type="continuous">
     <parent link="base_link" />
     <child link="right_wheel" />
-    <origin xyz="0.20 -0.225 0" rpy="${pi/2} 0 0" />
-    <axis xyz="0 0 1" />
+    <origin xyz="0.0 -0.175 0" rpy="${pi/2} 0 0" />
+    <axis xyz="0 0 -1" />
   </joint>
   <link name="right_wheel">
     <visual>
       <geometry>
-        <cylinder radius="0.1" length="0.05" />
+        <cylinder radius="0.05" length="0.04" />
       </geometry>
       <material name="blue" />
@@ -81,21 +87,24 @@
     <collision>
       <geometry>
-        <cylinder radius="0.1" length="0.05" />
+        <cylinder radius="0.05" length="0.04" />
       </geometry>
     </collision>
-    <xacro:inertial_cylinder mass="0.1" length="0.05" radius="0.1">
+    <xacro:inertial_cylinder mass="0.1" length="0.04" radius="0.05">
       <origin xyz="0 0 0" rpy="0 0 0" />
     </xacro:inertial_cylinder>
   </link>
+  <gazebo reference="right_wheel">
+    <material>Gazebo/Blue</material>
+  </gazebo>
   <!-- Caster wheels -->
-  <joint name="caster_wheel_1_joint" type="fixed">
+  <joint name="caster_wheel_joint" type="fixed">
     <parent link="chassis" />
-    <child link="caster_wheel_1" />
-    <origin xyz="0.1 0.11 0" />
+    <child link="caster_wheel" />
+    <origin xyz="0.24 0.0 0" rpy="0 0 0" />
   </joint>
-  <link name="caster_wheel_1">
+  <link name="caster_wheel">
     <visual>
       <geometry>
-        <sphere radius="0.09" />
+        <sphere radius="0.05" />
       </geometry>
       <material name="black" />
@@ -103,84 +112,26 @@
     <collision>
       <geometry>
-        <sphere radius="0.09" />
+        <sphere radius="0.05" />
       </geometry>
     </collision>
-    <xacro:inertial_sphere mass="0.1" radius="0.09">
+    <xacro:inertial_sphere mass="0.1" radius="0.05">
       <origin xyz="0 0 0" rpy="0 0 0" />
     </xacro:inertial_sphere>
   </link>
-  <joint name="caster_wheel_2_joint" type="fixed">
-    <parent link="chassis" />
-    <child link="caster_wheel_2" />
-    <origin xyz="0.1 -0.11 0" />
-  </joint>
-  <link name="caster_wheel_2">
-    <visual>
-      <geometry>
-        <sphere radius="0.09" />
-      </geometry>
-      <material name="black" />
-    </visual>
-    <collision>
-      <geometry>
-        <sphere radius="0.09" />
-      </geometry>
-    </collision>
-    <xacro:inertial_sphere mass="0.1" radius="0.09">
-      <origin xyz="0 0 0" rpy="0 0 0" />
-    </xacro:inertial_sphere>
-  </link>
-  <joint name="base_caster_wheel_3_joint" type="fixed">
-    <parent link="base_link" />
-    <child link="caster_wheel_3" />
-    <origin xyz="0.4 0.11 0" rpy="0 0 0" />
-  </joint>
-  <link name="caster_wheel_3">
-    <visual>
-      <geometry>
-        <sphere radius="0.09" />
-      </geometry>
-      <material name="black" />
-    </visual>
-    <collision>
-      <geometry>
-        <sphere radius="0.09" />
-      </geometry>
-    </collision>
-    <xacro:inertial_sphere mass="0.1" radius="0.09">
-      <origin xyz="0 0 0" rpy="0 0 0" />
-    </xacro:inertial_sphere>
-  </link>
-  <joint name="base_caster_wheel_4_joint" type="fixed">
-    <parent link="base_link" />
-    <child link="caster_wheel_4" />
-    <origin xyz="0.4 -0.11 0" rpy="0 0 0" />
-  </joint>
-  <link name="caster_wheel_4">
-    <visual>
-      <geometry>
-        <sphere radius="0.09" />
-      </geometry>
-      <material name="black" />
-    </visual>
-    <collision>
-      <geometry>
-        <sphere radius="0.09" />
-      </geometry>
-    </collision>
-    <xacro:inertial_sphere mass="0.1" radius="0.09">
-      <origin xyz="0 0 0" rpy="0 0 0" />
-    </xacro:inertial_sphere>
-  </link>
+  <gazebo reference="caster_wheel">
+    <material>Gazebo/Black</material>
+    <mu1 value="0.001"/>
+    <mu2 value="0.001"/>
+  </gazebo>
   <!-- LiDAR Tower -->
   <joint name="base_LiDAR_Tower_joint" type="fixed">
     <parent link="chassis" />
     <child link="LiDAR_Tower" />
-    <origin xyz="0.2 0.0 0.275" rpy="0 0 0" />
+    <origin xyz="0.12 0.0 0.18" rpy="0 0 0" />
   </joint>
   <link name="LiDAR_Tower">
     <visual>
       <geometry>
-        <box size="0.085 0.085 0.15" />
+        <box size="0.030 0.030 0.08" />
       </geometry>
       <material name="orange" />
@@ -188,34 +139,40 @@
     <collision>
       <geometry>
-        <box size="0.085 0.085 0.15" />
+        <box size="0.030 0.030 0.08" />
       </geometry>
     </collision>
-    <xacro:inertial_box mass="0.1" x="0.085" y="0.085" z="0.15">
+    <xacro:inertial_box mass="0.1" x="0.030" y="0.030" z="0.08">
       <origin xyz="0 0 0" rpy="0 0 0" />
     </xacro:inertial_box>
   </link>
+  <gazebo reference="LiDAR_Tower">
+    <material>Gazebo/Orange</material>
+  </gazebo>
   <!-- LiDAR Sensor -->
   <joint name="LiDAR_Tower_to_LiDAR_joint" type="fixed">
     <parent link="LiDAR_Tower" />
     <child link="LiDAR" />
-    <origin xyz="0 0 0" rpy="0 0 0" />
+    <origin xyz="0 0 0.044" rpy="0 0 0" />
   </joint>
   <link name="LiDAR">
     <visual>
       <geometry>
-        <cylinder radius="0.05" length="0.02" />
+        <cylinder radius="0.02" length="0.008" />
       </geometry>
-      <origin xyz="0 0 0.085" rpy="0 0 0" />
+      <origin xyz="0.0 0 0.0" rpy="0 0 0" />
       <material name="black" />
     </visual>
     <collision>
       <geometry>
-        <cylinder radius="0.05" length="0.02" />
+        <cylinder radius="0.025" length="0.005" />
       </geometry>
-      <origin xyz="0 0 0.085" rpy="0 0 0" />
+      <origin xyz="0 0 0.0" rpy="0 0 0" />
     </collision>
-    <xacro:inertial_cylinder mass="0.1" length="0.02" radius="0.05">
+    <xacro:inertial_cylinder mass="0.1" length="0.005" radius="0.025">
       <origin xyz="0 0 0" rpy="0 0 0" />
     </xacro:inertial_cylinder>
   </link>
+  <gazebo reference="LiDAR">
+    <material>Gazebo/Black</material>
+  </gazebo>
 </robot>
